File: kb-db/kb-db.sch (KiCad schematic (older format))
At the start: 12 parts, among them J1 Conn_01x04

Commit message: Ground components to USB ground
Parts:
- USB1: symbol Type-C:HRO-TYPE-C-31-M-12 -> kb-db-rescue:HRO-TYPE-C-31-M-12-Type-C
Connections:
- net Earth: now also C1.1, R5.1, USB1.13 (SHIELD); no longer C1.2, D1.1 (GND), R1.1, R2.1, R5.2
- net GND: now also C1.2, D1.1 (GND), R1.1, R2.1, R5.2
Changed lines of the file:
@@
 L power:Earth #PWR0106
 U 1 1 60896AC1
-P 2400 3800
-F 0 "#PWR0106" H 2400 3550 50  0001 C CNN
-F 1 "Earth" H 2400 3650 50  0001 C CNN
-F 2 "" H 2400 3800 50  0001 C CNN
-F 3 "~" H 2400 3800 50  0001 C CNN
-	1    2400 3800
-	1    0    0    -1
+P 2400 3400
+F 0 "#PWR0106" H 2400 3150 50  0001 C CNN
+F 1 "Earth" H 2400 3250 50  0001 C CNN
+F 2 "" H 2400 3400 50  0001 C CNN
+F 3 "~" H 2400 3400 50  0001 C CNN
+	1    2400 3400
+	0    -1   -1   0
 $EndComp
 $Comp
@@
 Text GLabel 4650 2750 1    50   Input ~ 0
 DBUS+
-$Comp
-L power:Earth #PWR0107
-U 1 1 608BCFA0
-P 4150 3250
-F 0 "#PWR0107" H 4150 3000 50  0001 C CNN
-F 1 "Earth" H 4150 3100 50  0001 C CNN
-F 2 "" H 4150 3250 50  0001 C CNN
-F 3 "~" H 4150 3250 50  0001 C CNN
-	1    4150 3250
-	1    0    0    -1
-$EndComp
 $Comp
 L power:VCC #PWR0108
@@
 Wire Wire Line
 	2550 2500 2400 2500
-$Comp
-L power:Earth #PWR0101
-U 1 1 609116B4
-P 2850 3100
-F 0 "#PWR0101" H 2850 2850 50  0001 C CNN
-F 1 "Earth" H 2850 2950 50  0001 C CNN
-F 2 "" H 2850 3100 50  0001 C CNN
-F 3 "~" H 2850 3100 50  0001 C CNN
-	1    2850 3100
-	1    0    0    -1
-$EndComp
-$Comp
-L power:Earth #PWR0102
-U 1 1 60911C23
-P 2850 2500
-F 0 "#PWR0102" H 2850 2250 50  0001 C CNN
-F 1 "Earth" H 2850 2350 50  0001 C CNN
-F 2 "" H 2850 2500 50  0001 C CNN
-F 3 "~" H 2850 2500 50  0001 C CNN
-	1    2850 2500
-	1    0    0    -1
-$EndComp
 Wire Wire Line
 	2750 3100 2850 3100
@@
 	2850 2200 2400 2200
 $Comp
-L Type-C:HRO-TYPE-C-31-M-12 USB1
+L kb-db-rescue:HRO-TYPE-C-31-M-12-Type-C USB1
 U 1 1 608E1765
 P 2300 2750
@@
 	1    0    0    -1
 $EndComp
+$Comp
+L power:GND #PWR0101
+U 1 1 61DFA349
+P 2850 2500
+F 0 "#PWR0101" H 2850 2250 50  0001 C CNN
+F 1 "GND" H 2855 2327 50  0000 C CNN
+F 2 "" H 2850 2500 50  0001 C CNN
+F 3 "" H 2850 2500 50  0001 C CNN
+	1    2850 2500
+	1    0    0    -1
+$EndComp
+$Comp
+L power:GND #PWR0102
+U 1 1 61DFA538
+P 2850 3100
+F 0 "#PWR0102" H 2850 2850 50  0001 C CNN
+F 1 "GND" H 2855 2927 50  0000 C CNN
+F 2 "" H 2850 3100 50  0001 C CNN
+F 3 "" H 2850 3100 50  0001 C CNN
+	1    2850 3100
+	1    0    0    -1
+$EndComp
+$Comp
+L power:GND #PWR0107
+U 1 1 61DFAAB9
+P 4150 3250
+F 0 "#PWR0107" H 4150 3000 50  0001 C CNN
+F 1 "GND" H 4155 3077 50  0000 C CNN
+F 2 "" H 4150 3250 50  0001 C CNN
+F 3 "" H 4150 3250 50  0001 C CNN
+	1    4150 3250
+	1    0    0    -1
+$EndComp
+Connection ~ 2400 3400
+$Comp
+L power:GND #PWR?
+U 1 1 61DFE648
+P 2400 3800
+F 0 "#PWR?" H 2400 3550 50  0001 C CNN
+F 1 "GND" H 2405 3627 50  0000 C CNN
+F 2 "" H 2400 3800 50  0001 C CNN
+F 3 "" H 2400 3800 50  0001 C CNN
+	1    2400 3800
+	1    0    0    -1
+$EndComp
